Commit message: inmoov_description: new LinkForge export, estimated inertia, self-collision SRDF
Model (re-exported from Blender):
- corrected joint axes and limits (rothead, eyes, fingers, elbows), mimic
  multipliers on the finger joints (Mid 0.8, Tip 0.6)
- simplified collisions: head/jaw/wrists/upper torso as boxes, forearms and
  hips as light convex STL; forearm-hip clearance at rest 7 mm -> 31 mm, so
  torso twist/lean no longer collides the arms with the hips
- two decimated visual meshes (jaw, head part)

Inertia: LinkForge rounds to 6 decimals, which zeroes fingertip tensors, so
mass/COM/full tensor are estimated from convex hulls of the visual meshes
(23.0 kg weighed incl. 6.88 kg stand, servo masses per link, density fitted
to ~20% of solid PLA) and kept in scripts/inertia_estimate.{json,csv}.
xacrify_scale.py now scales LinkForge inertia by model_scale^2 and applies
the estimate in the same run (--inertia / --no-inertia);
claude_compute_inertia.py recomputes it, apply_inertia.py re-applies it.

SRDF: description/inmoov_i2.srdf disables 228 of 903 pairs (adjacent,
head/jaw in the neck assembly, within each hand); zero pose is
collision-free. scripts/selfcoll.py is the sampling behind it.

README: regeneration in one command, mass/inertia method, SRDF.

Co-Authored-By: Claude Opus 5.5 <noreply@anthropic.com>

File: src/inmoov_description/description/inmoov_i2.urdf.xacro (robot description, xacro)
@@ -1,17 +1,17 @@
 <?xml version="1.0"?>
 <!--
-  Robot: inmoov_i2
+  Robot: inmoov_i1
   Generated by: LinkForge v1.5.1
   https://github.com/arounamounchili/linkforge
-  Date: 2026-09-21 19:54:19
+  Date: 2026-09-28 13:06:23
 -->
-<robot xmlns:xacro="http://www.ros.org/wiki/xacro" name="inmoov_i2">
+<robot xmlns:xacro="http://www.ros.org/wiki/xacro" name="inmoov_i1">
   <xacro:include filename="properties.xacro"/>
   <!-- Links -->
   <link name="NewHead_origin">
     <inertial>
-      <origin xyz="${model_scale*-0.000287} ${model_scale*0.239048} ${model_scale*0.160328}" rpy="0 0 0" />
-      <mass value="1" />
-      <inertia ixx="0.166667" ixy="0" ixz="0" iyy="0.166667" iyz="0" izz="0.166667" />
+      <origin xyz="-0.000718754 0.0405926 0.0266657" rpy="0 0 0" />
+      <mass value="1.16403" />
+      <inertia ixx="0.00557075" ixy="2.87555e-05" ixz="-3.77771e-05" iyy="0.00432267" iyz="0.000422277" izz="0.00439655" />
     </inertial>
     <visual>
@@ -88,5 +88,5 @@
     </visual>
     <visual>
-      <origin xyz="0 ${model_scale*0.348292} ${model_scale*0.331793}" rpy="0 0 0" />
+      <origin xyz="0 ${model_scale*0.348255} ${model_scale*0.331722}" rpy="0 0 0" />
       <geometry>
         <mesh filename="package://inmoov_description/meshes/NewHead_origin_visual_12.obj" scale="${model_scale} ${model_scale} ${model_scale}"/>
@@ -94,7 +94,7 @@
     </visual>
     <collision>
-      <origin xyz="${model_scale*-0.000287} ${model_scale*0.239048} ${model_scale*0.160328}" rpy="0 0 0" />
-      <geometry>
-        <mesh filename="package://inmoov_description/meshes/NewHead_origin_collision.stl" scale="${model_scale} ${model_scale} ${model_scale}"/>
+      <origin xyz="${model_scale*-0.000287} ${model_scale*0.239048} ${model_scale*0.160326}" rpy="0 0 0" />
+      <geometry>
+        <box size="${model_scale*1.36807} ${model_scale*1.942163} ${model_scale*1.765046}" />
       </geometry>
     </collision>
@@ -102,22 +102,24 @@
   <link name="i01_head_neck_001_link">
     <inertial>
+      <origin xyz="0 0 0" rpy="0 0 0" />
       <mass value="0.001" />
-      <inertia ixx="0.000001" ixy="0" ixz="0" iyy="0.000001" iyz="0" izz="0.000001" />
+      <inertia ixx="1e-09" ixy="0" ixz="0" iyy="1e-09" iyz="0" izz="1e-09" />
     </inertial>
   </link>
   <link name="i01_head_rothead_link">
     <inertial>
+      <origin xyz="0 0 0" rpy="0 0 0" />
       <mass value="0.001" />
-      <inertia ixx="0.000001" ixy="0" ixz="0" iyy="0.000001" iyz="0" izz="0.000001" />
+      <inertia ixx="1e-09" ixy="0" ixz="0" iyy="1e-09" iyz="0" izz="1e-09" />
     </inertial>
   </link>
   <link name="i02_head_eyeAssembly_origin">
     <inertial>
+      <origin xyz="-0.000116191 0.0105577 0.0104041" rpy="0 0 0" />
+      <mass value="0.034567" />
+      <inertia ixx="1.89139e-05" ixy="-2.37666e-21" ixz="2.01922e-21" iyy="5.9733e-05" iyz="1.98908e-06" izz="7.53723e-05" />
+    </inertial>
+    <visual>
       <origin xyz="${model_scale*0.326424} ${model_scale*0.169968} ${model_scale*0.121922}" rpy="0 0 0" />
-      <mass value="1" />
-      <inertia ixx="0.166667" ixy="0" ixz="0" iyy="0.166667" iyz="0" izz="0.166667" />
-    </inertial>
-    <visual>
-      <origin xyz="${model_scale*0.326424} ${model_scale*0.169968} ${model_scale*0.121922}" rpy="0 0 0" />
       <geometry>
         <mesh filename="package://inmoov_description/meshes/i02_head_eyeAssembly_origin_visual_0.obj" scale="${model_scale} ${model_scale} ${model_scale}"/>
@@ -145,18 +147,18 @@
   <link name="i02_head_jaw">
     <inertial>
-      <origin xyz="${model_scale*0.029643} ${model_scale*-0.354937} ${model_scale*-0.338088}" rpy="0 0 0" />
-      <mass value="1" />
-      <inertia ixx="0.166667" ixy="0" ixz="0" iyy="0.166667" iyz="0" izz="0.166667" />
-    </inertial>
-    <visual>
+      <origin xyz="0.00354333 -0.0396645 -0.0389397" rpy="0 0 0" />
+      <mass value="0.184096" />
+      <inertia ixx="0.000365167" ixy="-1.25204e-08" ixz="-6.52799e-09" iyy="0.000315219" iyz="-0.000143197" izz="0.000401922" />
+    </inertial>
+    <visual>
+      <origin xyz="${model_scale*0.029642} ${model_scale*-0.354923} ${model_scale*-0.338125}" rpy="0 0 0" />
+      <geometry>
+        <mesh filename="package://inmoov_description/meshes/i02_head_jaw_visual.obj" scale="${model_scale} ${model_scale} ${model_scale}"/>
+      </geometry>
+    </visual>
+    <collision>
       <origin xyz="${model_scale*0.029643} ${model_scale*-0.354913} ${model_scale*-0.338088}" rpy="0 0 0" />
       <geometry>
-        <mesh filename="package://inmoov_description/meshes/i02_head_jaw_visual.obj" scale="${model_scale} ${model_scale} ${model_scale}"/>
-      </geometry>
-    </visual>
-    <collision>
-      <origin xyz="${model_scale*0.029643} ${model_scale*-0.354937} ${model_scale*-0.338088}" rpy="0 0 0" />
-      <geometry>
-        <mesh filename="package://inmoov_description/meshes/i02_head_jaw_collision.stl" scale="${model_scale} ${model_scale} ${model_scale}"/>
+        <box size="${model_scale*1.101785} ${model_scale*1.283938} ${model_scale*0.973624}" />
       </geometry>
     </collision>
@@ -164,10 +166,10 @@
   <link name="i02_head_left_bottom_eyelid">
     <inertial>
+      <origin xyz="0.00804798 0.0113245 0.00400674" rpy="0 0 0" />
+      <mass value="0.00215896" />
+      <inertia ixx="2.18181e-07" ixy="-2.09214e-10" ixz="-8.5547e-12" iyy="1.14316e-07" iyz="6.14053e-10" izz="2.36628e-07" />
+    </inertial>
+    <visual>
       <origin xyz="${model_scale*0.081482} ${model_scale*0.092716} ${model_scale*0.064869}" rpy="0 0 0" />
-      <mass value="1" />
-      <inertia ixx="0.166667" ixy="0" ixz="0" iyy="0.166667" iyz="0" izz="0.166667" />
-    </inertial>
-    <visual>
-      <origin xyz="${model_scale*0.081482} ${model_scale*0.092716} ${model_scale*0.064869}" rpy="0 0 0" />
       <geometry>
         <mesh filename="package://inmoov_description/meshes/i02_head_left_bottom_eyelid_visual.obj" scale="${model_scale} ${model_scale} ${model_scale}"/>
@@ -177,10 +179,10 @@
   <link name="i02_head_left_cheek">
     <inertial>
+      <origin xyz="-0.00441059 -0.0216591 0.0013121" rpy="0 0 0" />
+      <mass value="0.0010832" />
+      <inertia ixx="1.69851e-07" ixy="-1.58525e-08" ixz="-1.54332e-09" iyy="2.36973e-08" iyz="7.48542e-09" izz="1.63312e-07" />
+    </inertial>
+    <visual>
       <origin xyz="${model_scale*-0.040165} ${model_scale*-0.153606} ${model_scale*0.007623}" rpy="0 0 0" />
-      <mass value="1" />
-      <inertia ixx="0.166667" ixy="0" ixz="0" iyy="0.166667" iyz="0" izz="0.166667" />
-    </inertial>
-    <visual>
-      <origin xyz="${model_scale*-0.040165} ${model_scale*-0.153606} ${model_scale*0.007623}" rpy="0 0 0" />
       <geometry>
         <mesh filename="package://inmoov_description/meshes/i02_head_left_cheek_visual.obj" scale="${model_scale} ${model_scale} ${model_scale}"/>
@@ -190,10 +192,10 @@
   <link name="i02_head_left_eye_horizontal">
     <inertial>
+      <origin xyz="-5.79762e-05 3.68601e-05 0.00265856" rpy="0 0 0" />
+      <mass value="0.000218835" />
+      <inertia ixx="1.56627e-09" ixy="-4.06662e-16" ixz="-2.52704e-14" iyy="9.34356e-09" iyz="2.46461e-11" izz="8.90905e-09" />
+    </inertial>
+    <visual>
       <origin xyz="${model_scale*-0.000485} ${model_scale*0.000044} ${model_scale*0.021219}" rpy="0 0 0" />
-      <mass value="1" />
-      <inertia ixx="0.166667" ixy="0" ixz="0" iyy="0.166667" iyz="0" izz="0.166667" />
-    </inertial>
-    <visual>
-      <origin xyz="${model_scale*-0.000485} ${model_scale*0.000044} ${model_scale*0.021219}" rpy="0 0 0" />
       <geometry>
         <mesh filename="package://inmoov_description/meshes/i02_head_left_eye_horizontal_visual.obj" scale="${model_scale} ${model_scale} ${model_scale}"/>
@@ -203,10 +205,10 @@
   <link name="i02_head_left_eye_vertical">
     <inertial>
+      <origin xyz="0.00213399 -0.0110728 0.000162328" rpy="0 0 0" />
+      <mass value="0.00561855" />
+      <inertia ixx="5.67536e-07" ixy="-5.80653e-10" ixz="1.49738e-08" iyy="5.3184e-07" iyz="2.7221e-10" izz="4.43697e-07" />
+    </inertial>
+    <visual>
       <origin xyz="${model_scale*-0.006014} ${model_scale*-0.093547} ${model_scale*0.001745}" rpy="3.141593 0 -1.570796" />
-      <mass value="1" />
-      <inertia ixx="0.166667" ixy="0" ixz="0" iyy="0.166667" iyz="0" izz="0.166667" />
-    </inertial>
-    <visual>
-      <origin xyz="${model_scale*-0.006014} ${model_scale*-0.093547} ${model_scale*0.001745}" rpy="3.141593 0 -1.570796" />
       <geometry>
         <mesh filename="package://inmoov_description/meshes/i02_head_left_eye_vertical_visual_0.obj" scale="${model_scale} ${model_scale} ${model_scale}"/>
@@ -240,10 +242,10 @@
   <link name="i02_head_left_eyebrow">
     <inertial>
+      <origin xyz="-0.0041037 -0.0056254 -0.00268787" rpy="0 0 0" />
+      <mass value="0.00241719" />
+      <inertia ixx="1.84901e-07" ixy="-8.53661e-08" ixz="2.04682e-08" iyy="2.6364e-07" iyz="1.11302e-08" izz="2.65682e-07" />
+    </inertial>
+    <visual>
       <origin xyz="${model_scale*-0.027981} ${model_scale*-0.037003} ${model_scale*-0.011673}" rpy="0 0 0" />
-      <mass value="1" />
-      <inertia ixx="0.166667" ixy="0" ixz="0" iyy="0.166667" iyz="0" izz="0.166667" />
-    </inertial>
-    <visual>
-      <origin xyz="${model_scale*-0.027981} ${model_scale*-0.037003} ${model_scale*-0.011673}" rpy="0 0 0" />
       <geometry>
         <mesh filename="package://inmoov_description/meshes/i02_head_left_eyebrow_visual.obj" scale="${model_scale} ${model_scale} ${model_scale}"/>
@@ -253,10 +255,10 @@
   <link name="i02_head_left_forehead">
     <inertial>
+      <origin xyz="0.00263627 0.00116021 -0.0120839" rpy="0 0 0" />
+      <mass value="0.00116402" />
+      <inertia ixx="1.20427e-07" ixy="-1.05031e-08" ixz="-2.63629e-08" iyy="1.54918e-07" iyz="-2.92519e-08" izz="6.06357e-08" />
+    </inertial>
+    <visual>
       <origin xyz="${model_scale*0.047329} ${model_scale*0.00672} ${model_scale*-0.132858}" rpy="0 0 0" />
-      <mass value="1" />
-      <inertia ixx="0.166667" ixy="0" ixz="0" iyy="0.166667" iyz="0" izz="0.166667" />
-    </inertial>
-    <visual>
-      <origin xyz="${model_scale*0.047329} ${model_scale*0.00672} ${model_scale*-0.132858}" rpy="0 0 0" />
       <geometry>
         <mesh filename="package://inmoov_description/meshes/i02_head_left_forehead_visual.obj" scale="${model_scale} ${model_scale} ${model_scale}"/>
@@ -266,10 +268,10 @@
   <link name="i02_head_left_top_eyelid">
     <inertial>
+      <origin xyz="-0.00829504 0.0111823 0.00403154" rpy="0 0 0" />
+      <mass value="0.00213019" />
+      <inertia ixx="2.09825e-07" ixy="1.83386e-10" ixz="-1.86533e-10" iyy="1.11888e-07" iyz="7.81562e-10" izz="2.26715e-07" />
+    </inertial>
+    <visual>
       <origin xyz="${model_scale*-0.082558} ${model_scale*0.09134} ${model_scale*0.064944}" rpy="0 0 0" />
-      <mass value="1" />
-      <inertia ixx="0.166667" ixy="0" ixz="0" iyy="0.166667" iyz="0" izz="0.166667" />
-    </inertial>
-    <visual>
-      <origin xyz="${model_scale*-0.082558} ${model_scale*0.09134} ${model_scale*0.064944}" rpy="0 0 0" />
       <geometry>
         <mesh filename="package://inmoov_description/meshes/i02_head_left_top_eyelid_visual.obj" scale="${model_scale} ${model_scale} ${model_scale}"/>
@@ -279,10 +281,10 @@
   <link name="i02_head_right_bottom_eyelid">
     <inertial>
+      <origin xyz="-0.00804798 0.0113245 0.00400674" rpy="0 0 0" />
+      <mass value="0.00215896" />
+      <inertia ixx="2.18181e-07" ixy="2.09222e-10" ixz="8.55812e-12" iyy="1.14316e-07" iyz="6.14054e-10" izz="2.36628e-07" />
+    </inertial>
+    <visual>
       <origin xyz="${model_scale*-0.081482} ${model_scale*0.092716} ${model_scale*0.064869}" rpy="0 0 0" />
-      <mass value="1" />
-      <inertia ixx="0.166667" ixy="0" ixz="0" iyy="0.166667" iyz="0" izz="0.166667" />
-    </inertial>
-    <visual>
-      <origin xyz="${model_scale*-0.081482} ${model_scale*0.092716} ${model_scale*0.064869}" rpy="0 0 0" />
       <geometry>
         <mesh filename="package://inmoov_description/meshes/i02_head_right_bottom_eyelid_visual.obj" scale="${model_scale} ${model_scale} ${model_scale}"/>
@@ -292,10 +294,10 @@
   <link name="i02_head_right_cheek">
     <inertial>
+      <origin xyz="0.00444838 -0.0216947 0.00119238" rpy="0 0 0" />
+      <mass value="0.0010832" />
+      <inertia ixx="1.69851e-07" ixy="1.58525e-08" ixz="1.54332e-09" iyy="2.36973e-08" iyz="7.48543e-09" izz="1.63312e-07" />
+    </inertial>
+    <visual>
       <origin xyz="${model_scale*0.040481} ${model_scale*-0.153904} ${model_scale*0.006622}" rpy="0 0 0" />
-      <mass value="1" />
-      <inertia ixx="0.166667" ixy="0" ixz="0" iyy="0.166667" iyz="0" izz="0.166667" />
-    </inertial>
-    <visual>
-      <origin xyz="${model_scale*0.040481} ${model_scale*-0.153904} ${model_scale*0.006622}" rpy="0 0 0" />
       <geometry>
         <mesh filename="package://inmoov_description/meshes/i02_head_right_cheek_visual.obj" scale="${model_scale} ${model_scale} ${model_scale}"/>
@@ -305,10 +307,10 @@
   <link name="i02_head_right_eye_horizontal">
     <inertial>
+      <origin xyz="5.79759e-05 3.68602e-05 0.00265856" rpy="0 0 0" />
+      <mass value="0.000218835" />
+      <inertia ixx="1.56627e-09" ixy="3.728e-16" ixz="2.54617e-14" iyy="9.34356e-09" iyz="2.4646e-11" izz="8.90905e-09" />
+    </inertial>
+    <visual>
       <origin xyz="${model_scale*0.000485} ${model_scale*0.000044} ${model_scale*0.021219}" rpy="0 0 0" />
-      <mass value="1" />
-      <inertia ixx="0.166667" ixy="0" ixz="0" iyy="0.166667" iyz="0" izz="0.166667" />
-    </inertial>
-    <visual>
-      <origin xyz="${model_scale*0.000485} ${model_scale*0.000044} ${model_scale*0.021219}" rpy="0 0 0" />
       <geometry>
         <mesh filename="package://inmoov_description/meshes/i02_head_right_eye_horizontal_visual.obj" scale="${model_scale} ${model_scale} ${model_scale}"/>
@@ -318,10 +320,10 @@
   <link name="i02_head_right_eye_vertical">
     <inertial>
+      <origin xyz="-0.00213399 0.0110719 -0.000162403" rpy="0 0 0" />
+      <mass value="0.00561855" />
+      <inertia ixx="5.67537e-07" ixy="-6.18983e-10" ixz="1.49704e-08" iyy="5.3184e-07" iyz="2.73675e-10" izz="4.43697e-07" />
+    </inertial>
+    <visual>
       <origin xyz="${model_scale*0.006014} ${model_scale*0.093547} ${model_scale*-0.001745}" rpy="0 0 -1.570796" />
-      <mass value="1" />
-      <inertia ixx="0.166667" ixy="0" ixz="0" iyy="0.166667" iyz="0" izz="0.166667" />
-    </inertial>
-    <visual>
-      <origin xyz="${model_scale*0.006014} ${model_scale*0.093547} ${model_scale*-0.001745}" rpy="0 0 -1.570796" />
       <geometry>
         <mesh filename="package://inmoov_description/meshes/i02_head_right_eye_vertical_visual_0.obj" scale="${model_scale} ${model_scale} ${model_scale}"/>
@@ -355,10 +357,10 @@
   <link name="i02_head_right_eyebrow">
     <inertial>
+      <origin xyz="0.00352856 -0.00370672 -0.00283611" rpy="0 0 0" />
+      <mass value="0.00258038" />
+      <inertia ixx="1.97011e-07" ixy="9.85765e-08" ixz="-2.90851e-08" iyy="3.07647e-07" iyz="1.37277e-08" izz="3.12151e-07" />
+    </inertial>
+    <visual>
       <origin xyz="${model_scale*0.019185} ${model_scale*-0.02342} ${model_scale*-0.011101}" rpy="0 0 0" />
-      <mass value="1" />
-      <inertia ixx="0.166667" ixy="0" ixz="0" iyy="0.166667" iyz="0" izz="0.166667" />
-    </inertial>
-    <visual>
-      <origin xyz="${model_scale*0.019185} ${model_scale*-0.02342} ${model_scale*-0.011101}" rpy="0 0 0" />
       <geometry>
         <mesh filename="package://inmoov_description/meshes/i02_head_right_eyebrow_visual.obj" scale="${model_scale} ${model_scale} ${model_scale}"/>
@@ -368,10 +370,10 @@
   <link name="i02_head_right_forehead">
     <inertial>
+      <origin xyz="-0.00263679 0.00116097 -0.0120824" rpy="0 0 0" />
+      <mass value="0.0011639" />
+      <inertia ixx="1.20392e-07" ixy="1.04987e-08" ixz="2.63537e-08" iyy="1.54885e-07" iyz="-2.92386e-08" izz="6.06255e-08" />
+    </inertial>
+    <visual>
       <origin xyz="${model_scale*-0.047329} ${model_scale*0.006778} ${model_scale*-0.132858}" rpy="0 0 0" />
-      <mass value="1" />
-      <inertia ixx="0.166667" ixy="0" ixz="0" iyy="0.166667" iyz="0" izz="0.166667" />
-    </inertial>
-    <visual>
-      <origin xyz="${model_scale*-0.047329} ${model_scale*0.006778} ${model_scale*-0.132858}" rpy="0 0 0" />
       <geometry>
         <mesh filename="package://inmoov_description/meshes/i02_head_right_forehead_visual.obj" scale="${model_scale} ${model_scale} ${model_scale}"/>
@@ -381,10 +383,10 @@
   <link name="i02_head_right_top_eyelid">
     <inertial>
+      <origin xyz="0.00829504 0.0111823 0.00403166" rpy="0 0 0" />
+      <mass value="0.00213019" />
+      <inertia ixx="2.09825e-07" ixy="-1.83396e-10" ixz="1.86533e-10" iyy="1.11888e-07" iyz="7.81563e-10" izz="2.26715e-07" />
+    </inertial>
+    <visual>
       <origin xyz="${model_scale*0.082558} ${model_scale*0.09134} ${model_scale*0.064945}" rpy="0 0 0" />
-      <mass value="1" />
-      <inertia ixx="0.166667" ixy="0" ixz="0" iyy="0.166667" iyz="0" izz="0.166667" />
-    </inertial>
-    <visual>
-      <origin xyz="${model_scale*0.082558} ${model_scale*0.09134} ${model_scale*0.064945}" rpy="0 0 0" />
       <geometry>
         <mesh filename="package://inmoov_description/meshes/i02_head_right_top_eyelid_visual.obj" scale="${model_scale} ${model_scale} ${model_scale}"/>
@@ -394,10 +396,10 @@
   <link name="i02_head_upper_lip">
     <inertial>
+      <origin xyz="0.0124013 -0.0308619 -0.0103012" rpy="0 0 0" />
+      <mass value="0.00435545" />
+      <inertia ixx="6.50928e-07" ixy="1.20692e-07" ixz="3.82743e-08" iyy="5.52123e-07" iyz="-1.34159e-07" izz="6.13437e-07" />
+    </inertial>
+    <visual>
       <origin xyz="${model_scale*0.127577} ${model_scale*-0.195387} ${model_scale*-0.112136}" rpy="0 0 0" />
-      <mass value="1" />
-      <inertia ixx="0.166667" ixy="0" ixz="0" iyy="0.166667" iyz="0" izz="0.166667" />
-    </inertial>
-    <visual>
-      <origin xyz="${model_scale*0.127577} ${model_scale*-0.195387} ${model_scale*-0.112136}" rpy="0 0 0" />
       <geometry>
         <mesh filename="package://inmoov_description/meshes/i02_head_upper_lip_visual.obj" scale="${model_scale} ${model_scale} ${model_scale}"/>
@@ -407,16 +409,16 @@
   <link name="i02_leftHand_ThumbMid">
     <inertial>
+      <origin xyz="0.0147526 -0.0128298 -0.000764153" rpy="0 0 0" />
+      <mass value="0.00555816" />
+      <inertia ixx="8.98565e-07" ixy="5.57166e-07" ixz="4.69106e-08" iyy="9.70967e-07" iyz="-5.14022e-08" izz="1.4978e-06" />
+    </inertial>
+    <visual>
+      <origin xyz="${model_scale*0.108091} ${model_scale*-0.105144} ${model_scale*-0.009741}" rpy="0 0 0" />
+      <geometry>
+        <mesh filename="package://inmoov_description/meshes/i02_leftHand_ThumbMid_visual.obj" scale="${model_scale} ${model_scale} ${model_scale}"/>
+      </geometry>
+    </visual>
+    <collision>
       <origin xyz="${model_scale*0.108091} ${model_scale*-0.105144} ${model_scale*-0.009742}" rpy="0 0 0" />
-      <mass value="1" />
-      <inertia ixx="0.166667" ixy="0" ixz="0" iyy="0.166667" iyz="0" izz="0.166667" />
-    </inertial>
-    <visual>
-      <origin xyz="${model_scale*0.108091} ${model_scale*-0.105144} ${model_scale*-0.009741}" rpy="0 0 0" />
-      <geometry>
-        <mesh filename="package://inmoov_description/meshes/i02_leftHand_ThumbMid_visual.obj" scale="${model_scale} ${model_scale} ${model_scale}"/>
-      </geometry>
-    </visual>
-    <collision>
-      <origin xyz="${model_scale*0.108091} ${model_scale*-0.105144} ${model_scale*-0.009742}" rpy="0 0 0" />
       <geometry>
         <mesh filename="package://inmoov_description/meshes/i02_leftHand_ThumbMid_collision.stl" scale="${model_scale} ${model_scale} ${model_scale}"/>
@@ -426,16 +428,16 @@
   <link name="i02_leftHand_ThumbTip">
     <inertial>
+      <origin xyz="0.00988169 -0.0140168 -0.00273774" rpy="0 0 0" />
+      <mass value="0.00342062" />
+      <inertia ixx="5.2478e-07" ixy="2.35701e-07" ixz="4.04439e-08" iyy="3.28382e-07" iyz="-5.82495e-08" izz="6.6944e-07" />
+    </inertial>
+    <visual>
+      <origin xyz="${model_scale*0.088894} ${model_scale*-0.115974} ${model_scale*-0.024371}" rpy="0 0 0" />
+      <geometry>
+        <mesh filename="package://inmoov_description/meshes/i02_leftHand_ThumbTip_visual.obj" scale="${model_scale} ${model_scale} ${model_scale}"/>
+      </geometry>
+    </visual>
+    <collision>
       <origin xyz="${model_scale*0.088894} ${model_scale*-0.115974} ${model_scale*-0.024438}" rpy="0 0 0" />
-      <mass value="1" />
-      <inertia ixx="0.166667" ixy="0" ixz="0" iyy="0.166667" iyz="0" izz="0.166667" />
-    </inertial>
-    <visual>
-      <origin xyz="${model_scale*0.088894} ${model_scale*-0.115974} ${model_scale*-0.024371}" rpy="0 0 0" />
-      <geometry>
-        <mesh filename="package://inmoov_description/meshes/i02_leftHand_ThumbTip_visual.obj" scale="${model_scale} ${model_scale} ${model_scale}"/>
-      </geometry>
-    </visual>
-    <collision>
-      <origin xyz="${model_scale*0.088894} ${model_scale*-0.115974} ${model_scale*-0.024438}" rpy="0 0 0" />
       <geometry>
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