Commit message: inmoov_description: drop stray left-hand meshes, recompute inertia
The left wrist link carried leftover parts (a 45k-vertex mesh, four
duplicate 2041-vertex pieces and two small ones) that the right wrist
doesn't have; the right wrist also lost one 25-vertex piece. Both wrists
now consist of the same five parts.

Since the inertia estimate comes from the visual meshes, it was recomputed:
left wrist 182 -> 168 g (now equal to the right one), hand with fingers
232 -> 218 g, other links within 0.5% (fitted density 242.6 -> 242.8
kg/m^3). Zero pose still collision-free, SRDF unchanged.

The .mtl files only change their header comment (source file renamed to
inmoov_i2.blend). New .blend in Git LFS.

Co-Authored-By: Claude Opus 5.5 <noreply@anthropic.com>

File: src/inmoov_description/description/inmoov_i2.urdf.xacro (robot description, xacro)
@@ -4,5 +4,5 @@
   Generated by: LinkForge v1.5.1
   https://github.com/arounamounchili/linkforge
-  Date: 2026-09-28 13:06:23
+  Date: 2026-09-28 17:02:50
 -->
 <robot xmlns:xacro="http://www.ros.org/wiki/xacro" name="inmoov_i2">
@@ -12,6 +12,6 @@
     <inertial>
       <origin xyz="-0.000718754 0.0405926 0.0266657" rpy="0 0 0" />
-      <mass value="1.16403" />
-      <inertia ixx="0.00557075" ixy="2.87555e-05" ixz="-3.77771e-05" iyy="0.00432267" iyz="0.000422277" izz="0.00439655" />
+      <mass value="1.1651" />
+      <inertia ixx="0.00557588" ixy="2.8782e-05" ixz="-3.78119e-05" iyy="0.00432665" iyz="0.000422665" izz="0.0044006" />
     </inertial>
     <visual>
@@ -117,6 +117,6 @@
     <inertial>
       <origin xyz="-0.000116191 0.0105577 0.0104041" rpy="0 0 0" />
-      <mass value="0.034567" />
-      <inertia ixx="1.89139e-05" ixy="-2.37666e-21" ixz="2.01922e-21" iyy="5.9733e-05" iyz="1.98908e-06" izz="7.53723e-05" />
+      <mass value="0.0346037" />
+      <inertia ixx="1.8934e-05" ixy="-2.37918e-21" ixz="2.02136e-21" iyy="5.97964e-05" iyz="1.99119e-06" izz="7.54523e-05" />
     </inertial>
     <visual>
@@ -148,6 +148,6 @@
     <inertial>
       <origin xyz="0.00354333 -0.0396645 -0.0389397" rpy="0 0 0" />
-      <mass value="0.184096" />
-      <inertia ixx="0.000365167" ixy="-1.25204e-08" ixz="-6.52799e-09" iyy="0.000315219" iyz="-0.000143197" izz="0.000401922" />
+      <mass value="0.184291" />
+      <inertia ixx="0.000365555" ixy="-1.25337e-08" ixz="-6.53492e-09" iyy="0.000315554" iyz="-0.000143349" izz="0.000402349" />
     </inertial>
     <visual>
@@ -167,6 +167,6 @@
     <inertial>
       <origin xyz="0.00804798 0.0113245 0.00400674" rpy="0 0 0" />
-      <mass value="0.00215896" />
-      <inertia ixx="2.18181e-07" ixy="-2.09214e-10" ixz="-8.5547e-12" iyy="1.14316e-07" iyz="6.14053e-10" izz="2.36628e-07" />
+      <mass value="0.00216126" />
+      <inertia ixx="2.18413e-07" ixy="-2.09436e-10" ixz="-8.56379e-12" iyy="1.14437e-07" iyz="6.14705e-10" izz="2.36879e-07" />
     </inertial>
     <visual>
@@ -180,6 +180,6 @@
     <inertial>
       <origin xyz="-0.00441059 -0.0216591 0.0013121" rpy="0 0 0" />
-      <mass value="0.0010832" />
-      <inertia ixx="1.69851e-07" ixy="-1.58525e-08" ixz="-1.54332e-09" iyy="2.36973e-08" iyz="7.48542e-09" izz="1.63312e-07" />
+      <mass value="0.00108435" />
+      <inertia ixx="1.70031e-07" ixy="-1.58694e-08" ixz="-1.54496e-09" iyy="2.37224e-08" iyz="7.49337e-09" izz="1.63485e-07" />
     </inertial>
     <visual>
@@ -193,6 +193,6 @@
     <inertial>
       <origin xyz="-5.79762e-05 3.68601e-05 0.00265856" rpy="0 0 0" />
-      <mass value="0.000218835" />
-      <inertia ixx="1.56627e-09" ixy="-4.06662e-16" ixz="-2.52704e-14" iyy="9.34356e-09" iyz="2.46461e-11" izz="8.90905e-09" />
+      <mass value="0.000219067" />
+      <inertia ixx="1.56794e-09" ixy="-4.07094e-16" ixz="-2.52972e-14" iyy="9.35348e-09" iyz="2.46722e-11" izz="8.91851e-09" />
     </inertial>
     <visual>
@@ -206,6 +206,6 @@
     <inertial>
       <origin xyz="0.00213399 -0.0110728 0.000162328" rpy="0 0 0" />
-      <mass value="0.00561855" />
-      <inertia ixx="5.67536e-07" ixy="-5.80653e-10" ixz="1.49738e-08" iyy="5.3184e-07" iyz="2.7221e-10" izz="4.43697e-07" />
+      <mass value="0.00562452" />
+      <inertia ixx="5.68139e-07" ixy="-5.81269e-10" ixz="1.49897e-08" iyy="5.32405e-07" iyz="2.72499e-10" izz="4.44168e-07" />
     </inertial>
     <visual>
@@ -243,6 +243,6 @@
     <inertial>
       <origin xyz="-0.0041037 -0.0056254 -0.00268787" rpy="0 0 0" />
-      <mass value="0.00241719" />
-      <inertia ixx="1.84901e-07" ixy="-8.53661e-08" ixz="2.04682e-08" iyy="2.6364e-07" iyz="1.11302e-08" izz="2.65682e-07" />
+      <mass value="0.00241976" />
+      <inertia ixx="1.85098e-07" ixy="-8.54567e-08" ixz="2.04899e-08" iyy="2.6392e-07" iyz="1.1142e-08" izz="2.65964e-07" />
     </inertial>
     <visual>
@@ -256,6 +256,6 @@
     <inertial>
       <origin xyz="0.00263627 0.00116021 -0.0120839" rpy="0 0 0" />
-      <mass value="0.00116402" />
-      <inertia ixx="1.20427e-07" ixy="-1.05031e-08" ixz="-2.63629e-08" iyy="1.54918e-07" iyz="-2.92519e-08" izz="6.06357e-08" />
+      <mass value="0.00116526" />
+      <inertia ixx="1.20555e-07" ixy="-1.05142e-08" ixz="-2.63909e-08" iyy="1.55082e-07" iyz="-2.92829e-08" izz="6.07001e-08" />
     </inertial>
     <visual>
@@ -269,6 +269,6 @@
     <inertial>
       <origin xyz="-0.00829504 0.0111823 0.00403154" rpy="0 0 0" />
-      <mass value="0.00213019" />
-      <inertia ixx="2.09825e-07" ixy="1.83386e-10" ixz="-1.86533e-10" iyy="1.11888e-07" iyz="7.81562e-10" izz="2.26715e-07" />
+      <mass value="0.00213245" />
+      <inertia ixx="2.10048e-07" ixy="1.83581e-10" ixz="-1.86732e-10" iyy="1.12007e-07" iyz="7.82392e-10" izz="2.26956e-07" />
     </inertial>
     <visual>
@@ -282,6 +282,6 @@
     <inertial>
       <origin xyz="-0.00804798 0.0113245 0.00400674" rpy="0 0 0" />
-      <mass value="0.00215896" />
-      <inertia ixx="2.18181e-07" ixy="2.09222e-10" ixz="8.55812e-12" iyy="1.14316e-07" iyz="6.14054e-10" izz="2.36628e-07" />
+      <mass value="0.00216126" />
+      <inertia ixx="2.18413e-07" ixy="2.09444e-10" ixz="8.5672e-12" iyy="1.14437e-07" iyz="6.14706e-10" izz="2.36879e-07" />
     </inertial>
     <visual>
@@ -295,6 +295,6 @@
     <inertial>
       <origin xyz="0.00444838 -0.0216947 0.00119238" rpy="0 0 0" />
-      <mass value="0.0010832" />
-      <inertia ixx="1.69851e-07" ixy="1.58525e-08" ixz="1.54332e-09" iyy="2.36973e-08" iyz="7.48543e-09" izz="1.63312e-07" />
+      <mass value="0.00108435" />
+      <inertia ixx="1.70031e-07" ixy="1.58694e-08" ixz="1.54496e-09" iyy="2.37224e-08" iyz="7.49338e-09" izz="1.63485e-07" />
     </inertial>
     <visual>
@@ -308,6 +308,6 @@
     <inertial>
       <origin xyz="5.79759e-05 3.68602e-05 0.00265856" rpy="0 0 0" />
-      <mass value="0.000218835" />
-      <inertia ixx="1.56627e-09" ixy="3.728e-16" ixz="2.54617e-14" iyy="9.34356e-09" iyz="2.4646e-11" izz="8.90905e-09" />
+      <mass value="0.000219067" />
+      <inertia ixx="1.56794e-09" ixy="3.73196e-16" ixz="2.54887e-14" iyy="9.35348e-09" iyz="2.46722e-11" izz="8.91851e-09" />
     </inertial>
     <visual>
@@ -321,6 +321,6 @@
     <inertial>
       <origin xyz="-0.00213399 0.0110719 -0.000162403" rpy="0 0 0" />
-      <mass value="0.00561855" />
-      <inertia ixx="5.67537e-07" ixy="-6.18983e-10" ixz="1.49704e-08" iyy="5.3184e-07" iyz="2.73675e-10" izz="4.43697e-07" />
+      <mass value="0.00562452" />
+      <inertia ixx="5.6814e-07" ixy="-6.19641e-10" ixz="1.49863e-08" iyy="5.32404e-07" iyz="2.73966e-10" izz="4.44168e-07" />
     </inertial>
     <visual>
@@ -358,6 +358,6 @@
     <inertial>
       <origin xyz="0.00352856 -0.00370672 -0.00283611" rpy="0 0 0" />
-      <mass value="0.00258038" />
-      <inertia ixx="1.97011e-07" ixy="9.85765e-08" ixz="-2.90851e-08" iyy="3.07647e-07" iyz="1.37277e-08" izz="3.12151e-07" />
+      <mass value="0.00258313" />
+      <inertia ixx="1.97221e-07" ixy="9.86812e-08" ixz="-2.9116e-08" iyy="3.07973e-07" iyz="1.37422e-08" izz="3.12482e-07" />
     </inertial>
     <visual>
@@ -371,6 +371,6 @@
     <inertial>
       <origin xyz="-0.00263679 0.00116097 -0.0120824" rpy="0 0 0" />
-      <mass value="0.0011639" />
-      <inertia ixx="1.20392e-07" ixy="1.04987e-08" ixz="2.63537e-08" iyy="1.54885e-07" iyz="-2.92386e-08" izz="6.06255e-08" />
+      <mass value="0.00116513" />
+      <inertia ixx="1.20519e-07" ixy="1.05098e-08" ixz="2.63817e-08" iyy="1.55049e-07" iyz="-2.92697e-08" izz="6.06899e-08" />
     </inertial>
     <visual>
@@ -384,6 +384,6 @@
     <inertial>
       <origin xyz="0.00829504 0.0111823 0.00403166" rpy="0 0 0" />
-      <mass value="0.00213019" />
-      <inertia ixx="2.09825e-07" ixy="-1.83396e-10" ixz="1.86533e-10" iyy="1.11888e-07" iyz="7.81563e-10" izz="2.26715e-07" />
+      <mass value="0.00213245" />
+      <inertia ixx="2.10048e-07" ixy="-1.83591e-10" ixz="1.86731e-10" iyy="1.12007e-07" iyz="7.82393e-10" izz="2.26956e-07" />
     </inertial>
     <visual>
@@ -397,6 +397,6 @@
     <inertial>
       <origin xyz="0.0124013 -0.0308619 -0.0103012" rpy="0 0 0" />
-      <mass value="0.00435545" />
-      <inertia ixx="6.50928e-07" ixy="1.20692e-07" ixz="3.82743e-08" iyy="5.52123e-07" iyz="-1.34159e-07" izz="6.13437e-07" />
+      <mass value="0.00436007" />
+      <inertia ixx="6.51619e-07" ixy="1.20821e-07" ixz="3.83149e-08" iyy="5.52709e-07" iyz="-1.34301e-07" izz="6.14088e-07" />
     </inertial>
     <visual>
@@ -410,6 +410,6 @@
     <inertial>
       <origin xyz="0.0147526 -0.0128298 -0.000764153" rpy="0 0 0" />
-      <mass value="0.00555816" />
-      <inertia ixx="8.98565e-07" ixy="5.57166e-07" ixz="4.69106e-08" iyy="9.70967e-07" iyz="-5.14022e-08" izz="1.4978e-06" />
+      <mass value="0.00556406" />
+      <inertia ixx="8.99519e-07" ixy="5.57757e-07" ixz="4.69604e-08" iyy="9.71998e-07" iyz="-5.14567e-08" izz="1.49939e-06" />
     </inertial>
     <visual>
@@ -429,6 +429,6 @@
     <inertial>
       <origin xyz="0.00988169 -0.0140168 -0.00273774" rpy="0 0 0" />
-      <mass value="0.00342062" />
-      <inertia ixx="5.2478e-07" ixy="2.35701e-07" ixz="4.04439e-08" iyy="3.28382e-07" iyz="-5.82495e-08" izz="6.6944e-07" />
+      <mass value="0.00342425" />
+      <inertia ixx="5.25337e-07" ixy="2.35951e-07" ixz="4.04869e-08" iyy="3.28731e-07" iyz="-5.83114e-08" izz="6.70151e-07" />
     </inertial>
     <visual>
@@ -448,6 +448,6 @@
     <inertial>
       <origin xyz="0.00131022 -0.0062803 -0.0129446" rpy="0 0 0" />
-      <mass value="0.00292044" />
-      <inertia ixx="4.707e-07" ixy="4.11764e-09" ixz="1.52108e-08" iyy="3.96772e-07" iyz="-1.37095e-07" izz="2.06695e-07" />
+      <mass value="0.00292354" />
+      <inertia ixx="4.712e-07" ixy="4.12201e-09" ixz="1.5227e-08" iyy="3.97194e-07" iyz="-1.3724e-07" izz="2.06915e-07" />
     </inertial>
     <visual>
@@ -467,6 +467,6 @@
     <inertial>
       <origin xyz="0.000708628 -0.00785698 -0.0148538" rpy="0 0 0" />
-      <mass value="0.00516345" />
-      <inertia ixx="1.33103e-06" ixy="1.21417e-08" ixz="5.60559e-08" iyy="1.11813e-06" iyz="-4.01435e-07" izz="5.30535e-07" />
+      <mass value="0.00516894" />
+      <inertia ixx="1.33245e-06" ixy="1.21546e-08" ixz="5.61154e-08" iyy="1.11932e-06" iyz="-4.01861e-07" izz="5.31098e-07" />
     </inertial>
     <visual>
@@ -486,6 +486,6 @@
     <inertial>
       <origin xyz="0.00109558 -0.00534797 -0.0119621" rpy="0 0 0" />
-      <mass value="0.00271215" />
-      <inertia ixx="3.39421e-07" ixy="1.18332e-08" ixz="1.10256e-08" iyy="3.08824e-07" iyz="-8.102e-08" izz="1.68628e-07" />
+      <mass value="0.00271503" />
+      <inertia ixx="3.39782e-07" ixy="1.18458e-08" ixz="1.10373e-08" iyy="3.09152e-07" iyz="-8.1106e-08" izz="1.68807e-07" />
     </inertial>
     <visual>
@@ -505,6 +505,6 @@
     <inertial>
       <origin xyz="0.000478318 -0.0056054 -0.0132517" rpy="0 0 0" />
-      <mass value="0.00292043" />
-      <inertia ixx="4.71332e-07" ixy="-5.42752e-09" ixz="-3.54658e-09" iyy="4.07708e-07" iyz="-1.28952e-07" izz="1.95126e-07" />
+      <mass value="0.00292353" />
+      <inertia ixx="4.71832e-07" ixy="-5.43329e-09" ixz="-3.55035e-09" iyy="4.08141e-07" iyz="-1.29089e-07" izz="1.95334e-07" />
     </inertial>
     <visual>
@@ -524,6 +524,6 @@
     <inertial>
       <origin xyz="-0.000522032 -0.00713112 -0.015021" rpy="0 0 0" />
-      <mass value="0.00516273" />
-      <inertia ixx="1.33389e-06" ixy="-1.61441e-08" ixz="-5.51595e-10" iyy="1.14989e-06" iyz="-3.76591e-07" izz="4.9543e-07" />
+      <mass value="0.00516821" />
+      <inertia ixx="1.33531e-06" ixy="-1.61612e-08" ixz="-5.52181e-10" iyy="1.15111e-06" iyz="-3.7699e-07" izz="4.95956e-07" />
     </inertial>
     <visual>
@@ -543,6 +543,6 @@
     <inertial>
       <origin xyz="0.000475776 -0.00558965 -0.0133367" rpy="0 0 0" />
-      <mass value="0.00221884" />
-      <inertia ixx="3.20767e-07" ixy="2.95772e-09" ixz="1.20457e-09" iyy="2.85423e-07" iyz="-8.76887e-08" izz="1.16608e-07" />
+      <mass value="0.0022212" />
+      <inertia ixx="3.21107e-07" ixy="2.96086e-09" ixz="1.20585e-09" iyy="2.85727e-07" iyz="-8.77819e-08" izz="1.16732e-07" />
     </inertial>
     <visual>
@@ -562,6 +562,6 @@
     <inertial>
       <origin xyz="-0.00167063 -0.00461326 -0.0136405" rpy="0 0 0" />
-      <mass value="0.00292043" />
-      <inertia ixx="4.63553e-07" ixy="-2.06145e-08" ixz="-4.66035e-08" iyy="4.3041e-07" iyz="-1.04868e-07" izz="1.80204e-07" />
+      <mass value="0.00292353" />
+      <inertia ixx="4.64045e-07" ixy="-2.06363e-08" ixz="-4.6653e-08" iyy="4.30867e-07" iyz="-1.04979e-07" izz="1.80395e-07" />
     </inertial>
     <visual>
@@ -581,6 +581,6 @@
     <inertial>
       <origin xyz="-0.00314023 -0.00565968 -0.0149356" rpy="0 0 0" />
-      <mass value="0.00516345" />
-      <inertia ixx="1.31326e-06" ixy="-6.09829e-08" ixz="-1.30466e-07" iyy="1.21623e-06" iyz="-3.03453e-07" izz="4.50204e-07" />
+      <mass value="0.00516894" />
+      <inertia ixx="1.31466e-06" ixy="-6.10477e-08" ixz="-1.30605e-07" iyy="1.21753e-06" iyz="-3.03775e-07" izz="4.50682e-07" />
     </inertial>
     <visual>
@@ -600,6 +600,6 @@
     <inertial>
       <origin xyz="-0.00107632 -0.00317951 -0.0104729" rpy="0 0 0" />
-      <mass value="0.00182093" />
-      <inertia ixx="1.91141e-07" ixy="-3.38646e-09" ixz="-1.51332e-08" iyy="1.82589e-07" iyz="-3.6646e-08" izz="7.70718e-08" />
+      <mass value="0.00182287" />
+      <inertia ixx="1.91344e-07" ixy="-3.39006e-09" ixz="-1.51493e-08" iyy="1.82783e-07" iyz="-3.66849e-08" izz="7.71536e-08" />
     </inertial>
     <visual>
@@ -619,6 +619,6 @@
     <inertial>
       <origin xyz="-0.00057257 -0.00517935 -0.0136954" rpy="0 0 0" />
-      <mass value="0.00292043" />
-      <inertia ixx="4.68848e-07" ixy="-1.43941e-08" ixz="-2.58085e-08" iyy="4.1984e-07" iyz="-1.17394e-07" izz="1.85479e-07" />
+      <mass value="0.00292354" />
+      <inertia ixx="4.69345e-07" ixy="-1.44094e-08" ixz="-2.58359e-08" iyy="4.20286e-07" iyz="-1.17519e-07" izz="1.85676e-07" />
     </inertial>
     <visual>
@@ -638,6 +638,6 @@
     <inertial>
       <origin xyz="-0.00159384 -0.00615466 -0.0152816" rpy="0 0 0" />
-      <mass value="0.00516345" />
-      <inertia ixx="1.32796e-06" ixy="-4.26596e-08" ixz="-6.76613e-08" iyy="1.18551e-06" iyz="-3.41422e-07" izz="4.66231e-07" />
+      <mass value="0.00516894" />
+      <inertia ixx="1.32937e-06" ixy="-4.27049e-08" ixz="-6.77332e-08" iyy="1.18677e-06" iyz="-3.41785e-07" izz="4.66726e-07" />
     </inertial>
     <visual>
@@ -657,6 +657,6 @@
     <inertial>
       <origin xyz="-0.000154814 -0.00354383 -0.0104197" rpy="0 0 0" />
-      <mass value="0.00182093" />
-      <inertia ixx="1.92606e-07" ixy="-1.21964e-09" ixz="-7.13645e-09" iyy="1.79076e-07" iyz="-4.1536e-08" izz="7.912e-08" />
+      <mass value="0.00182287" />
+      <inertia ixx="1.9281e-07" ixy="-1.22093e-09" ixz="-7.14403e-09" iyy="1.79266e-07" iyz="-4.15801e-08" izz="7.9204e-08" />
     </inertial>
     <visual>
@@ -676,6 +676,6 @@
     <inertial>
       <origin xyz="-0.0146851 -0.0130156 -0.00108614" rpy="0 0 0" />
-      <mass value="0.00555817" />
-      <inertia ixx="8.98571e-07" ixy="-5.57169e-07" ixz="-4.69107e-08" iyy="9.70972e-07" iyz="-5.14023e-08" izz="1.49781e-06" />
+      <mass value="0.00556408" />
+      <inertia ixx="8.99525e-07" ixy="-5.57761e-07" ixz="-4.69606e-08" iyy="9.72003e-07" iyz="-5.14569e-08" izz="1.4994e-06" />
     </inertial>
     <visual>
@@ -695,6 +695,6 @@
     <inertial>
       <origin xyz="-0.00996755 -0.0140526 -0.00269519" rpy="0 0 0" />
-      <mass value="0.00342063" />
-      <inertia ixx="5.24782e-07" ixy="-2.35701e-07" ixz="-4.04439e-08" iyy="3.28383e-07" iyz="-5.82497e-08" izz="6.69442e-07" />
+      <mass value="0.00342426" />
+      <inertia ixx="5.25339e-07" ixy="-2.35952e-07" ixz="-4.04869e-08" iyy="3.28731e-07" iyz="-5.83115e-08" izz="6.70153e-07" />
     </inertial>
     <visual>
@@ -714,6 +714,6 @@
     <inertial>
       <origin xyz="-0.00136069 -0.00629575 -0.013173" rpy="0 0 0" />
-      <mass value="0.00292044" />
-      <inertia ixx="4.70701e-07" ixy="-4.11764e-09" ixz="-1.52109e-08" iyy="3.96773e-07" iyz="-1.37095e-07" izz="2.06695e-07" />
+      <mass value="0.00292354" />
+      <inertia ixx="4.71201e-07" ixy="-4.12202e-09" ixz="-1.5227e-08" iyy="3.97195e-07" iyz="-1.37241e-07" izz="2.06915e-07" />
     </inertial>
     <visual>
@@ -733,6 +733,6 @@
     <inertial>
       <origin xyz="-0.000769622 -0.00800446 -0.0151004" rpy="0 0 0" />
-      <mass value="0.00516346" />
-      <inertia ixx="1.33104e-06" ixy="-1.21418e-08" ixz="-5.6056e-08" iyy="1.11814e-06" iyz="-4.01436e-07" izz="5.30536e-07" />
+      <mass value="0.00516895" />
+      <inertia ixx="1.33245e-06" ixy="-1.21546e-08" ixz="-5.61155e-08" iyy="1.11933e-06" iyz="-4.01863e-07" izz="5.311e-07" />
     </inertial>
     <visual>
@@ -752,6 +752,6 @@
     <inertial>
       <origin xyz="-0.00117202 -0.00540782 -0.0122147" rpy="0 0 0" />
-      <mass value="0.00271215" />
-      <inertia ixx="3.39422e-07" ixy="-1.18332e-08" ixz="-1.10255e-08" iyy="3.08824e-07" iyz="-8.102e-08" izz="1.68628e-07" />
+      <mass value="0.00271503" />
+      <inertia ixx="3.39782e-07" ixy="-1.18458e-08" ixz="-1.10372e-08" iyy="3.09152e-07" iyz="-8.11061e-08" izz="1.68807e-07" />
     </inertial>
     <visual>
@@ -771,6 +771,6 @@
     <inertial>
       <origin xyz="-0.00020147 -0.00570656 -0.0133627" rpy="0 0 0" />
-      <mass value="0.00292044" />
-      <inertia ixx="4.71334e-07" ixy="5.42755e-09" ixz="3.54647e-09" iyy="4.0771e-07" iyz="-1.28953e-07" izz="1.95127e-07" />
+      <mass value="0.00292354" />
+      <inertia ixx="4.71834e-07" ixy="5.43332e-09" ixz="3.55024e-09" iyy="4.08143e-07" iyz="-1.2909e-07" izz="1.95334e-07" />
     </inertial>
     <visual>
@@ -790,6 +790,6 @@
     <inertial>
       <origin xyz="0.000238311 -0.0071328 -0.0151598" rpy="0 0 0" />
-      <mass value="0.00516274" />
-      <inertia ixx="1.3339e-06" ixy="1.61443e-08" ixz="5.51667e-10" iyy="1.14989e-06" iyz="-3.76592e-07" izz="4.95432e-07" />
+      <mass value="0.00516822" />
+      <inertia ixx="1.33531e-06" ixy="1.61614e-08" ixz="5.52253e-10" iyy="1.15111e-06" iyz="-3.76992e-07" izz="4.95958e-07" />
     </inertial>
     <visual>
@@ -809,6 +809,6 @@
     <inertial>
       <origin xyz="-0.000600311 -0.00538527 -0.0132005" rpy="0 0 0" />
-      <mass value="0.00221885" />
-      <inertia ixx="3.20768e-07" ixy="-2.95775e-09" ixz="-1.20455e-09" iyy="2.85425e-07" iyz="-8.76891e-08" izz="1.16608e-07" />
+      <mass value="0.0022212" />
+      <inertia ixx="3.21109e-07" ixy="-2.9609e-09" ixz="-1.20583e-09" iyy="2.85728e-07" iyz="-8.77822e-08" izz="1.16732e-07" />
     </inertial>
     <visual>
@@ -828,6 +828,6 @@
     <inertial>
       <origin xyz="0.00149159 -0.00458601 -0.013729" rpy="0 0 0" />
-      <mass value="0.00292044" />
-      <inertia ixx="4.63554e-07" ixy="2.06145e-08" ixz="4.66036e-08" iyy="4.30411e-07" iyz="-1.04868e-07" izz="1.80204e-07" />
+      <mass value="0.00292354" />
+      <inertia ixx="4.64046e-07" ixy="2.06364e-08" ixz="4.66531e-08" iyy="4.30869e-07" iyz="-1.0498e-07" izz="1.80395e-07" />
     </inertial>
     <visual>
@@ -847,6 +847,6 @@
     <inertial>
       <origin xyz="0.0027934 -0.00578909 -0.0150138" rpy="0 0 0" />
-      <mass value="0.00516346" />
-      <inertia ixx="1.31327e-06" ixy="6.09831e-08" ixz="1.30467e-07" iyy="1.21624e-06" iyz="-3.03454e-07" izz="4.50205e-07" />
+      <mass value="0.00516895" />
+      <inertia ixx="1.31466e-06" ixy="6.10479e-08" ixz="1.30605e-07" iyy="1.21753e-06" iyz="-3.03776e-07" izz="4.50683e-07" />
     </inertial>
     <visual>
@@ -866,6 +866,6 @@
     <inertial>
       <origin xyz="0.000839267 -0.0033234 -0.0106647" rpy="0 0 0" />
-      <mass value="0.00182094" />
-      <inertia ixx="1.91142e-07" ixy="3.38646e-09" ixz="1.51333e-08" iyy="1.8259e-07" iyz="-3.66462e-08" izz="7.7072e-08" />
+      <mass value="0.00182287" />
+      <inertia ixx="1.91345e-07" ixy="3.39006e-09" ixz="1.51493e-08" iyy="1.82784e-07" iyz="-3.66851e-08" izz="7.71538e-08" />
     </inertial>
     <visual>
@@ -885,6 +885,6 @@
     <inertial>
       <origin xyz="0.000717644 -0.0051234 -0.0137816" rpy="0 0 0" />
-      <mass value="0.00292044" />
-      <inertia ixx="4.68849e-07" ixy="1.43942e-08" ixz="2.58087e-08" iyy="4.19841e-07" iyz="-1.17395e-07" izz="1.8548e-07" />
+      <mass value="0.00292354" />
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