Commit message: inmoov_description: new torso parts, OAK-D frames, model_scale 0.10604
- New LinkForge export: two new torso_y_link parts (visual_44..78
  renumbered), OAK-D frames oak_mount_link (fixed to torso_y_link, x
  forward) and oak_rgb_camera_optical_frame (ROS optical convention),
  ~1.30 m above the floor. New .blend in Git LFS.
- model_scale 0.1196 -> 0.10604, recalibrated against the physical robot:
  crown 1.81 m above the floor in the zero pose, stand included.
- Inertia estimate recomputed for the new scale and meshes (reproduced by
  claude_compute_inertia.py to 1e-16, notes in English): fitted density
  ~20% -> ~28% of solid PLA, total still 23.0 kg, all 65 tensors valid.
- Self-collisions unchanged (uniform scale): zero pose clean, SRDF as is.
- README / properties.xacro: new scale, OAK-D frames, and that the SI
  inertia must be recomputed after a scale change.

Co-Authored-By: Claude Opus 5.5 <noreply@anthropic.com>

File: src/inmoov_description/description/inmoov_i2.urdf.xacro (robot description, xacro)
@@ -4,5 +4,5 @@
   Generated by: LinkForge v1.5.1
   https://github.com/arounamounchili/linkforge
-  Date: 2026-09-28 17:02:50
+  Date: 2026-10-05 11:52:14
 -->
 <robot xmlns:xacro="http://www.ros.org/wiki/xacro" name="inmoov_i2">
@@ -11,7 +11,7 @@
   <link name="NewHead_origin">
     <inertial>
-      <origin xyz="-0.000718754 0.0405926 0.0266657" rpy="0 0 0" />
-      <mass value="1.1651" />
-      <inertia ixx="0.00557588" ixy="2.8782e-05" ixz="-3.78119e-05" iyy="0.00432665" iyz="0.000422665" izz="0.0044006" />
+      <origin xyz="-0.000637263 0.0359903 0.0236424" rpy="0 0 0" />
+      <mass value="1.17544" />
+      <inertia ixx="0.00442207" ixy="2.28261e-05" ixz="-2.99875e-05" iyy="0.00343134" iyz="0.000335203" izz="0.00348998" />
     </inertial>
     <visual>
@@ -116,7 +116,7 @@
   <link name="i02_head_eyeAssembly_origin">
     <inertial>
-      <origin xyz="-0.000116191 0.0105577 0.0104041" rpy="0 0 0" />
-      <mass value="0.0346037" />
-      <inertia ixx="1.8934e-05" ixy="-2.37918e-21" ixz="2.02136e-21" iyy="5.97964e-05" iyz="1.99119e-06" izz="7.54523e-05" />
+      <origin xyz="-0.000103018 0.00936068 0.0092245" rpy="0 0 0" />
+      <mass value="0.0349577" />
+      <inertia ixx="1.50363e-05" ixy="-1.68786e-21" ixz="-2.31569e-21" iyy="4.74867e-05" iyz="1.58128e-06" izz="5.99197e-05" />
     </inertial>
     <visual>
@@ -147,7 +147,7 @@
   <link name="i02_head_jaw">
     <inertial>
-      <origin xyz="0.00354333 -0.0396645 -0.0389397" rpy="0 0 0" />
-      <mass value="0.184291" />
-      <inertia ixx="0.000365555" ixy="-1.25337e-08" ixz="-6.53492e-09" iyy="0.000315554" iyz="-0.000143349" izz="0.000402349" />
+      <origin xyz="0.00314159 -0.0351675 -0.0345248" rpy="0 0 0" />
+      <mass value="0.186176" />
+      <inertia ixx="0.000290301" ixy="-9.9535e-09" ixz="-5.18964e-09" iyy="0.000250594" iyz="-0.000113839" izz="0.000319521" />
     </inertial>
     <visual>
@@ -166,7 +166,7 @@
   <link name="i02_head_left_bottom_eyelid">
     <inertial>
-      <origin xyz="0.00804798 0.0113245 0.00400674" rpy="0 0 0" />
-      <mass value="0.00216126" />
-      <inertia ixx="2.18413e-07" ixy="-2.09436e-10" ixz="-8.56379e-12" iyy="1.14437e-07" iyz="6.14705e-10" izz="2.36879e-07" />
+      <origin xyz="0.00713552 0.0100406 0.00355246" rpy="0 0 0" />
+      <mass value="0.00218336" />
+      <inertia ixx="1.7345e-07" ixy="-1.66321e-10" ixz="-6.80085e-12" iyy="9.08793e-08" iyz="4.88162e-10" izz="1.88115e-07" />
     </inertial>
     <visual>
@@ -179,7 +179,7 @@
   <link name="i02_head_left_cheek">
     <inertial>
-      <origin xyz="-0.00441059 -0.0216591 0.0013121" rpy="0 0 0" />
-      <mass value="0.00108435" />
-      <inertia ixx="1.70031e-07" ixy="-1.58694e-08" ixz="-1.54496e-09" iyy="2.37224e-08" iyz="7.49337e-09" izz="1.63485e-07" />
+      <origin xyz="-0.00391053 -0.0192034 0.00116334" rpy="0 0 0" />
+      <mass value="0.00109544" />
+      <inertia ixx="1.35028e-07" ixy="-1.26025e-08" ixz="-1.22691e-09" iyy="1.88389e-08" iyz="5.95078e-09" izz="1.2983e-07" />
     </inertial>
     <visual>
@@ -192,7 +192,7 @@
   <link name="i02_head_left_eye_horizontal">
     <inertial>
-      <origin xyz="-5.79762e-05 3.68601e-05 0.00265856" rpy="0 0 0" />
-      <mass value="0.000219067" />
-      <inertia ixx="1.56794e-09" ixy="-4.07094e-16" ixz="-2.52972e-14" iyy="9.35348e-09" iyz="2.46722e-11" izz="8.91851e-09" />
+      <origin xyz="-5.1403e-05 3.2681e-05 0.00235714" rpy="0 0 0" />
+      <mass value="0.000221308" />
+      <inertia ixx="1.24516e-09" ixy="-3.2329e-16" ixz="-2.00895e-14" iyy="7.42797e-09" iyz="1.95932e-11" izz="7.08254e-09" />
     </inertial>
     <visual>
@@ -205,7 +205,7 @@
   <link name="i02_head_left_eye_vertical">
     <inertial>
-      <origin xyz="0.00213399 -0.0110728 0.000162328" rpy="0 0 0" />
-      <mass value="0.00562452" />
-      <inertia ixx="5.68139e-07" ixy="-5.81269e-10" ixz="1.49897e-08" iyy="5.32405e-07" iyz="2.72499e-10" izz="4.44168e-07" />
+      <origin xyz="0.00189204 -0.00981736 0.000143924" rpy="0 0 0" />
+      <mass value="0.00568205" />
+      <inertia ixx="4.51182e-07" ixy="-4.61609e-10" ixz="1.19039e-08" iyy="4.22804e-07" iyz="2.16403e-10" izz="3.52731e-07" />
     </inertial>
     <visual>
@@ -242,7 +242,7 @@
   <link name="i02_head_left_eyebrow">
     <inertial>
-      <origin xyz="-0.0041037 -0.0056254 -0.00268787" rpy="0 0 0" />
-      <mass value="0.00241976" />
-      <inertia ixx="1.85098e-07" ixy="-8.54567e-08" ixz="2.04899e-08" iyy="2.6392e-07" iyz="1.1142e-08" izz="2.65964e-07" />
+      <origin xyz="-0.00363843 -0.0049876 -0.00238313" rpy="0 0 0" />
+      <mass value="0.00244451" />
+      <inertia ixx="1.46994e-07" ixy="-6.78646e-08" ixz="1.62719e-08" iyy="2.0959e-07" iyz="8.84834e-09" izz="2.11213e-07" />
     </inertial>
     <visual>
@@ -255,7 +255,7 @@
   <link name="i02_head_left_forehead">
     <inertial>
-      <origin xyz="0.00263627 0.00116021 -0.0120839" rpy="0 0 0" />
-      <mass value="0.00116526" />
-      <inertia ixx="1.20555e-07" ixy="-1.05142e-08" ixz="-2.63909e-08" iyy="1.55082e-07" iyz="-2.92829e-08" izz="6.07001e-08" />
+      <origin xyz="0.00233738 0.00102867 -0.0107139" rpy="0 0 0" />
+      <mass value="0.00117718" />
+      <inertia ixx="9.57375e-08" ixy="-8.34978e-09" ixz="-2.09581e-08" iyy="1.23157e-07" iyz="-2.32548e-08" izz="4.82044e-08" />
     </inertial>
     <visual>
@@ -268,7 +268,7 @@
   <link name="i02_head_left_top_eyelid">
     <inertial>
-      <origin xyz="-0.00829504 0.0111823 0.00403154" rpy="0 0 0" />
-      <mass value="0.00213245" />
-      <inertia ixx="2.10048e-07" ixy="1.83581e-10" ixz="-1.86732e-10" iyy="1.12007e-07" iyz="7.82392e-10" izz="2.26956e-07" />
+      <origin xyz="-0.00735456 0.00991449 0.00357446" rpy="0 0 0" />
+      <mass value="0.00215427" />
+      <inertia ixx="1.66807e-07" ixy="1.45789e-10" ixz="-1.48291e-10" iyy="8.89489e-08" iyz="6.21329e-10" izz="1.80235e-07" />
     </inertial>
     <visual>
@@ -281,7 +281,7 @@
   <link name="i02_head_right_bottom_eyelid">
     <inertial>
-      <origin xyz="-0.00804798 0.0113245 0.00400674" rpy="0 0 0" />
-      <mass value="0.00216126" />
-      <inertia ixx="2.18413e-07" ixy="2.09444e-10" ixz="8.5672e-12" iyy="1.14437e-07" iyz="6.14706e-10" izz="2.36879e-07" />
+      <origin xyz="-0.00713552 0.0100406 0.00355246" rpy="0 0 0" />
+      <mass value="0.00218336" />
+      <inertia ixx="1.7345e-07" ixy="1.66328e-10" ixz="6.80356e-12" iyy="9.08794e-08" iyz="4.88163e-10" izz="1.88115e-07" />
     </inertial>
     <visual>
@@ -294,7 +294,7 @@
   <link name="i02_head_right_cheek">
     <inertial>
-      <origin xyz="0.00444838 -0.0216947 0.00119238" rpy="0 0 0" />
-      <mass value="0.00108435" />
-      <inertia ixx="1.70031e-07" ixy="1.58694e-08" ixz="1.54496e-09" iyy="2.37224e-08" iyz="7.49338e-09" izz="1.63485e-07" />
+      <origin xyz="0.00394403 -0.019235 0.00105719" rpy="0 0 0" />
+      <mass value="0.00109544" />
+      <inertia ixx="1.35029e-07" ixy="1.26025e-08" ixz="1.22691e-09" iyy="1.88389e-08" iyz="5.95079e-09" izz="1.2983e-07" />
     </inertial>
     <visual>
@@ -307,7 +307,7 @@
   <link name="i02_head_right_eye_horizontal">
     <inertial>
-      <origin xyz="5.79759e-05 3.68602e-05 0.00265856" rpy="0 0 0" />
-      <mass value="0.000219067" />
-      <inertia ixx="1.56794e-09" ixy="3.73196e-16" ixz="2.54887e-14" iyy="9.35348e-09" iyz="2.46722e-11" izz="8.91851e-09" />
+      <origin xyz="5.14027e-05 3.26811e-05 0.00235714" rpy="0 0 0" />
+      <mass value="0.000221308" />
+      <inertia ixx="1.24516e-09" ixy="2.96369e-16" ixz="2.02416e-14" iyy="7.42797e-09" iyz="1.95932e-11" izz="7.08254e-09" />
     </inertial>
     <visual>
@@ -320,7 +320,7 @@
   <link name="i02_head_right_eye_vertical">
     <inertial>
-      <origin xyz="-0.00213399 0.0110719 -0.000162403" rpy="0 0 0" />
-      <mass value="0.00562452" />
-      <inertia ixx="5.6814e-07" ixy="-6.19641e-10" ixz="1.49863e-08" iyy="5.32404e-07" iyz="2.73966e-10" izz="4.44168e-07" />
+      <origin xyz="-0.00189204 0.0098166 -0.00014399" rpy="0 0 0" />
+      <mass value="0.00568205" />
+      <inertia ixx="4.51182e-07" ixy="-4.92081e-10" ixz="1.19012e-08" iyy="4.22804e-07" iyz="2.17567e-10" izz="3.52732e-07" />
     </inertial>
     <visual>
@@ -357,7 +357,7 @@
   <link name="i02_head_right_eyebrow">
     <inertial>
-      <origin xyz="0.00352856 -0.00370672 -0.00283611" rpy="0 0 0" />
-      <mass value="0.00258313" />
-      <inertia ixx="1.97221e-07" ixy="9.86812e-08" ixz="-2.9116e-08" iyy="3.07973e-07" iyz="1.37422e-08" izz="3.12482e-07" />
+      <origin xyz="0.0031285 -0.00328646 -0.00251456" rpy="0 0 0" />
+      <mass value="0.00260955" />
+      <inertia ixx="1.56621e-07" ixy="7.83667e-08" ixz="-2.31222e-08" iyy="2.44574e-07" iyz="1.09133e-08" izz="2.48155e-07" />
     </inertial>
     <visual>
@@ -370,7 +370,7 @@
   <link name="i02_head_right_forehead">
     <inertial>
-      <origin xyz="-0.00263679 0.00116097 -0.0120824" rpy="0 0 0" />
-      <mass value="0.00116513" />
-      <inertia ixx="1.20519e-07" ixy="1.05098e-08" ixz="2.63817e-08" iyy="1.55049e-07" iyz="-2.92697e-08" izz="6.06899e-08" />
+      <origin xyz="-0.00233783 0.00102934 -0.0107125" rpy="0 0 0" />
+      <mass value="0.00117705" />
+      <inertia ixx="9.57093e-08" ixy="8.34629e-09" ixz="2.09508e-08" iyy="1.23131e-07" iyz="-2.32442e-08" izz="4.81963e-08" />
     </inertial>
     <visual>
@@ -383,7 +383,7 @@
   <link name="i02_head_right_top_eyelid">
     <inertial>
-      <origin xyz="0.00829504 0.0111823 0.00403166" rpy="0 0 0" />
-      <mass value="0.00213245" />
-      <inertia ixx="2.10048e-07" ixy="-1.83591e-10" ixz="1.86731e-10" iyy="1.12007e-07" iyz="7.82393e-10" izz="2.26956e-07" />
+      <origin xyz="0.00735456 0.00991449 0.00357456" rpy="0 0 0" />
+      <mass value="0.00215427" />
+      <inertia ixx="1.66807e-07" ixy="-1.45797e-10" ixz="1.4829e-10" iyy="8.89489e-08" iyz="6.21329e-10" izz="1.80235e-07" />
     </inertial>
     <visual>
@@ -396,7 +396,7 @@
   <link name="i02_head_upper_lip">
     <inertial>
-      <origin xyz="0.0124013 -0.0308619 -0.0103012" rpy="0 0 0" />
-      <mass value="0.00436007" />
-      <inertia ixx="6.51619e-07" ixy="1.20821e-07" ixz="3.83149e-08" iyy="5.52709e-07" iyz="-1.34301e-07" izz="6.14088e-07" />
+      <origin xyz="0.0109952 -0.0273628 -0.00913327" rpy="0 0 0" />
+      <mass value="0.00440467" />
+      <inertia ixx="5.17477e-07" ixy="9.59484e-08" ixz="3.04274e-08" iyy="4.38929e-07" iyz="-1.06654e-07" izz="4.87672e-07" />
     </inertial>
     <visual>
@@ -409,7 +409,7 @@
   <link name="i02_leftHand_ThumbMid">
     <inertial>
-      <origin xyz="0.0147526 -0.0128298 -0.000764153" rpy="0 0 0" />
-      <mass value="0.00556406" />
-      <inertia ixx="8.99519e-07" ixy="5.57757e-07" ixz="4.69604e-08" iyy="9.71998e-07" iyz="-5.14567e-08" izz="1.49939e-06" />
+      <origin xyz="0.01308 -0.0113752 -0.000677515" rpy="0 0 0" />
+      <mass value="0.00562098" />
+      <inertia ixx="7.14344e-07" ixy="4.42937e-07" ixz="3.72931e-08" iyy="7.71903e-07" iyz="-4.08639e-08" izz="1.19073e-06" />
     </inertial>
     <visual>
@@ -428,7 +428,7 @@
   <link name="i02_leftHand_ThumbTip">
     <inertial>
-      <origin xyz="0.00988169 -0.0140168 -0.00273774" rpy="0 0 0" />
-      <mass value="0.00342425" />
-      <inertia ixx="5.25337e-07" ixy="2.35951e-07" ixz="4.04869e-08" iyy="3.28731e-07" iyz="-5.83114e-08" izz="6.70151e-07" />
+      <origin xyz="0.00876133 -0.0124276 -0.00242734" rpy="0 0 0" />
+      <mass value="0.00345928" />
+      <inertia ixx="4.17191e-07" ixy="1.87378e-07" ixz="3.21522e-08" iyy="2.61058e-07" iyz="-4.63074e-08" izz="5.32194e-07" />
     </inertial>
     <visual>
@@ -447,7 +447,7 @@
   <link name="i02_leftHand_indexMid">
     <inertial>
-      <origin xyz="0.00131022 -0.0062803 -0.0129446" rpy="0 0 0" />
-      <mass value="0.00292354" />
-      <inertia ixx="4.712e-07" ixy="4.12201e-09" ixz="1.5227e-08" iyy="3.97194e-07" iyz="-1.3724e-07" izz="2.06915e-07" />
+      <origin xyz="0.00116167 -0.00556826 -0.011477" rpy="0 0 0" />
+      <mass value="0.00295344" />
+      <inertia ixx="3.74199e-07" ixy="3.27345e-09" ixz="1.20923e-08" iyy="3.15428e-07" iyz="-1.08988e-07" izz="1.64319e-07" />
     </inertial>
     <visual>
@@ -466,7 +466,7 @@
   <link name="i02_leftHand_indexPhal">
     <inertial>
-      <origin xyz="0.000708628 -0.00785698 -0.0148538" rpy="0 0 0" />
-      <mass value="0.00516894" />
-      <inertia ixx="1.33245e-06" ixy="1.21546e-08" ixz="5.61154e-08" iyy="1.11932e-06" iyz="-4.01861e-07" izz="5.31098e-07" />
+      <origin xyz="0.000628285 -0.00696617 -0.0131698" rpy="0 0 0" />
+      <mass value="0.00522181" />
+      <inertia ixx="1.05815e-06" ixy="9.65245e-09" ixz="4.45635e-08" iyy="8.88898e-07" iyz="-3.19134e-07" izz="4.21766e-07" />
     </inertial>
     <visual>
@@ -485,7 +485,7 @@
   <link name="i02_leftHand_indexTip">
     <inertial>
-      <origin xyz="0.00109558 -0.00534797 -0.0119621" rpy="0 0 0" />
-      <mass value="0.00271503" />
-      <inertia ixx="3.39782e-07" ixy="1.18458e-08" ixz="1.10373e-08" iyy="3.09152e-07" iyz="-8.1106e-08" izz="1.68807e-07" />
+      <origin xyz="0.000971365 -0.00474163 -0.0106059" rpy="0 0 0" />
+      <mass value="0.0027428" />
+      <inertia ixx="2.69834e-07" ixy="9.40722e-09" ixz="8.76516e-09" iyy="2.4551e-07" iyz="-6.44095e-08" izz="1.34056e-07" />
     </inertial>
     <visual>
@@ -504,7 +504,7 @@
   <link name="i02_leftHand_majeureMid">
     <inertial>
-      <origin xyz="0.000478318 -0.0056054 -0.0132517" rpy="0 0 0" />
-      <mass value="0.00292353" />
-      <inertia ixx="4.71832e-07" ixy="-5.43329e-09" ixz="-3.55035e-09" iyy="4.08141e-07" iyz="-1.29089e-07" izz="1.95334e-07" />
+      <origin xyz="0.000424087 -0.00496987 -0.0117493" rpy="0 0 0" />
+      <mass value="0.00295344" />
+      <inertia ixx="3.74701e-07" ixy="-4.31479e-09" ixz="-2.81947e-09" iyy="3.24121e-07" iyz="-1.02515e-07" izz="1.55122e-07" />
     </inertial>
     <visual>
@@ -523,7 +523,7 @@
   <link name="i02_leftHand_majeurePhal">
     <inertial>
-      <origin xyz="-0.000522032 -0.00713112 -0.015021" rpy="0 0 0" />
-      <mass value="0.00516821" />
-      <inertia ixx="1.33531e-06" ixy="-1.61612e-08" ixz="-5.52181e-10" iyy="1.15111e-06" iyz="-3.7699e-07" izz="4.95956e-07" />
+      <origin xyz="-0.000462845 -0.00632261 -0.013318" rpy="0 0 0" />
+      <mass value="0.00522108" />
+      <inertia ixx="1.06042e-06" ixy="-1.28343e-08" ixz="-4.38509e-10" iyy="9.1414e-07" iyz="-2.99383e-07" izz="3.93859e-07" />
     </inertial>
     <visual>
@@ -542,7 +542,7 @@
   <link name="i02_leftHand_majeureTip">
     <inertial>
-      <origin xyz="0.000475776 -0.00558965 -0.0133367" rpy="0 0 0" />
-      <mass value="0.0022212" />
-      <inertia ixx="3.21107e-07" ixy="2.96086e-09" ixz="1.20585e-09" iyy="2.85727e-07" iyz="-8.77819e-08" izz="1.16732e-07" />
+      <origin xyz="0.000421834 -0.00495591 -0.0118246" rpy="0 0 0" />
+      <mass value="0.00224392" />
+      <inertia ixx="2.55004e-07" ixy="2.35134e-09" ixz="9.57613e-10" iyy="2.26907e-07" iyz="-6.97111e-08" izz="9.27012e-08" />
     </inertial>
     <visual>
@@ -561,7 +561,7 @@
   <link name="i02_leftHand_pinkyMid">
     <inertial>
-      <origin xyz="-0.00167063 -0.00461326 -0.0136405" rpy="0 0 0" />
-      <mass value="0.00292353" />
-      <inertia ixx="4.64045e-07" ixy="-2.06363e-08" ixz="-4.6653e-08" iyy="4.30867e-07" iyz="-1.04979e-07" izz="1.80395e-07" />
+      <origin xyz="-0.00148121 -0.00409022 -0.012094" rpy="0 0 0" />
+      <mass value="0.00295344" />
+      <inertia ixx="3.68517e-07" ixy="-1.63881e-08" ixz="-3.7049e-08" iyy="3.42169e-07" iyz="-8.3368e-08" izz="1.43259e-07" />
     </inertial>
     <visual>
@@ -580,7 +580,7 @@
   <link name="i02_leftHand_pinkyPhal">
     <inertial>
-      <origin xyz="-0.00314023 -0.00565968 -0.0149356" rpy="0 0 0" />
-      <mass value="0.00516894" />
-      <inertia ixx="1.31466e-06" ixy="-6.10477e-08" ixz="-1.30605e-07" iyy="1.21753e-06" iyz="-3.03775e-07" izz="4.50682e-07" />
+      <origin xyz="-0.00278419 -0.00501799 -0.0132423" rpy="0 0 0" />
+      <mass value="0.00522181" />
+      <inertia ixx="1.04402e-06" ixy="-4.84804e-08" ixz="-1.03718e-07" iyy="9.66886e-07" iyz="-2.4124e-07" izz="3.57904e-07" />
     </inertial>
     <visual>
@@ -599,7 +599,7 @@
   <link name="i02_leftHand_pinkyTip">
     <inertial>
-      <origin xyz="-0.00107632 -0.00317951 -0.0104729" rpy="0 0 0" />
-      <mass value="0.00182287" />
-      <inertia ixx="1.91344e-07" ixy="-3.39006e-09" ixz="-1.51493e-08" iyy="1.82783e-07" iyz="-3.66849e-08" izz="7.71536e-08" />
+      <origin xyz="-0.000954285 -0.00281903 -0.00928546" rpy="0 0 0" />
+      <mass value="0.00184151" />
+      <inertia ixx="1.51954e-07" ixy="-2.69218e-09" ixz="-1.20306e-08" iyy="1.45155e-07" iyz="-2.9133e-08" izz="6.12708e-08" />
     </inertial>
     <visual>
@@ -618,7 +618,7 @@
   <link name="i02_leftHand_ringFingerMid">
     <inertial>
-      <origin xyz="-0.00057257 -0.00517935 -0.0136954" rpy="0 0 0" />
-      <mass value="0.00292354" />
-      <inertia ixx="4.69345e-07" ixy="-1.44094e-08" ixz="-2.58359e-08" iyy="4.20286e-07" iyz="-1.17519e-07" izz="1.85676e-07" />
+      <origin xyz="-0.000507653 -0.00459213 -0.0121427" rpy="0 0 0" />
+      <mass value="0.00295344" />
+      <inertia ixx="3.72726e-07" ixy="-1.1443e-08" ixz="-2.05173e-08" iyy="3.33766e-07" iyz="-9.33265e-08" izz="1.47453e-07" />
     </inertial>
     <visual>
@@ -637,7 +637,7 @@
   <link name="i02_leftHand_ringFingerPhal">
     <inertial>
-      <origin xyz="-0.00159384 -0.00615466 -0.0152816" rpy="0 0 0" />
-      <mass value="0.00516894" />
-      <inertia ixx="1.32937e-06" ixy="-4.27049e-08" ixz="-6.77332e-08" iyy="1.18677e-06" iyz="-3.41785e-07" izz="4.66726e-07" />
+      <origin xyz="-0.00141313 -0.00545685 -0.013549" rpy="0 0 0" />
+      <mass value="0.00522181" />
+      <inertia ixx="1.05571e-06" ixy="-3.39137e-08" ixz="-5.37896e-08" iyy="9.42461e-07" iyz="-2.71425e-07" izz="3.70646e-07" />
     </inertial>
     <visual>
@@ -656,7 +656,7 @@
   <link name="i02_leftHand_ringFingerTip">
     <inertial>
-      <origin xyz="-0.000154814 -0.00354383 -0.0104197" rpy="0 0 0" />
-      <mass value="0.00182287" />
-      <inertia ixx="1.9281e-07" ixy="-1.22093e-09" ixz="-7.14403e-09" iyy="1.79266e-07" iyz="-4.15801e-08" izz="7.9204e-08" />
+      <origin xyz="-0.000137262 -0.00314204 -0.00923833" rpy="0 0 0" />
+      <mass value="0.00184151" />
+      <inertia ixx="1.53119e-07" ixy="-9.69592e-10" ixz="-5.67336e-09" iyy="1.42362e-07" iyz="-3.30204e-08" izz="6.2899e-08" />
     </inertial>
     <visual>
@@ -675,7 +675,7 @@
   <link name="i02_rightHand_ThumbMid">
     <inertial>
-      <origin xyz="-0.0146851 -0.0130156 -0.00108614" rpy="0 0 0" />
-      <mass value="0.00556408" />
-      <inertia ixx="8.99525e-07" ixy="-5.57761e-07" ixz="-4.69606e-08" iyy="9.72003e-07" iyz="-5.14569e-08" izz="1.4994e-06" />
+      <origin xyz="-0.0130201 -0.0115399 -0.000962992" rpy="0 0 0" />
+      <mass value="0.00562099" />
+      <inertia ixx="7.14349e-07" ixy="-4.4294e-07" ixz="-3.72933e-08" iyy="7.71906e-07" iyz="-4.0864e-08" izz="1.19073e-06" />
     </inertial>
     <visual>
@@ -694,7 +694,7 @@
   <link name="i02_rightHand_ThumbTip">
     <inertial>
-      <origin xyz="-0.00996755 -0.0140526 -0.00269519" rpy="0 0 0" />
-      <mass value="0.00342426" />
-      <inertia ixx="5.25339e-07" ixy="-2.35952e-07" ixz="-4.04869e-08" iyy="3.28731e-07" iyz="-5.83115e-08" izz="6.70153e-07" />
+      <origin xyz="-0.00883745 -0.0124594 -0.00238962" rpy="0 0 0" />
+      <mass value="0.00345929" />
+      <inertia ixx="4.17193e-07" ixy="-1.87379e-07" ixz="-3.21522e-08" iyy="2.61059e-07" iyz="-4.63075e-08" izz="5.32196e-07" />
     </inertial>
     <visual>
@@ -713,7 +713,7 @@
   <link name="i02_rightHand_indexMid">
     <inertial>
-      <origin xyz="-0.00136069 -0.00629575 -0.013173" rpy="0 0 0" />
-      <mass value="0.00292354" />
-      <inertia ixx="4.71201e-07" ixy="-4.12202e-09" ixz="-1.5227e-08" iyy="3.97195e-07" iyz="-1.37241e-07" izz="2.06915e-07" />
+      <origin xyz="-0.00120642 -0.00558195 -0.0116795" rpy="0 0 0" />
+      <mass value="0.00295345" />
+      <inertia ixx="3.742e-07" ixy="-3.27346e-09" ixz="-1.20924e-08" iyy="3.15428e-07" iyz="-1.08988e-07" izz="1.64319e-07" />
     </inertial>
     <visual>
@@ -732,7 +732,7 @@
   <link name="i02_rightHand_indexPhal">
     <inertial>
-      <origin xyz="-0.000769622 -0.00800446 -0.0151004" rpy="0 0 0" />
-      <mass value="0.00516895" />
-      <inertia ixx="1.33245e-06" ixy="-1.21546e-08" ixz="-5.61155e-08" iyy="1.11933e-06" iyz="-4.01863e-07" izz="5.311e-07" />
+      <origin xyz="-0.000682364 -0.00709693 -0.0133883" rpy="0 0 0" />
+      <mass value="0.00522182" />
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
File: src/inmoov_description/description/properties.xacro (robot description, xacro)
@@ -4,10 +4,12 @@
 units, not meters — every <origin xyz> and <mesh scale> in that file is
 written as ${model_scale*...} against this property.
-0.1196 is carried over from the old Sentience-Robotics inmoov_urdf
-properties.xacro, which calibrated it to a measured crown height of 1.80 m
-on the same underlying model. Re-check/recalibrate against the physical
-robot if it drifts after a fresh LinkForge export.
+0.10604 (2026-10-05) is recalibrated against the physical robot: in the zero
+pose the crown is 1.81 m above the floor, stand included. It replaced 0.1196,
+carried over from the old Sentience-Robotics inmoov_urdf properties.xacro.
+The mass/inertia estimate (scripts/inertia_estimate.json) is stored in SI
+units for this scale: after changing model_scale, recompute it with
+scripts/claude_compute_inertia.py and re-apply it.
 -->
 <robot xmlns:xacro="http://www.ros.org/wiki/xacro">
-  <xacro:property name="model_scale" value="0.1196"/>
+  <xacro:property name="model_scale" value="0.10604"/>
 </robot>
